File: AstralPool.kicad_sch (KiCad schematic)
At the start: 19 parts, among them J1 RJ12, J2 RJ12, J3 Header, J4 Conn_02x12_Counter_Clockwise, Q1 MMBT3904, U1 LM2678S-5.0/NOPB

Commit message: ### Changed - Rev 10 - moved C5 closer to U1 - Rev 10 - added via under U1 - Rev 10 - minor layout improvements.
Parts:
- D1, D2: value D 6TQ045S -> PMEG6010CEH,115
Changed lines of the file:
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@@
 	(title_block
 		(title "Connect 10 Controller")
-		(date "2026-02-17")
-		(rev "9")
+		(date "2026-02-18")
+		(rev "10")
 	)
 	(text "+5v"
@@
 			)
 		)
-		(property "Value" "D 6TQ045S"
+		(property "Value" "PMEG6010CEH,115"
 			(at 132.3975 53.34 0)
 			(effects
@@
 			)
 		)
-		(property "Value" "D 6TQ045S"
+		(property "Value" "PMEG6010CEH,115"
 			(at 80.01 83.5024 90)
 			(effects

Commit message: ### Changed - Rev 10 - Updated all part numbers and use MPN instead of PartNum
Parts:
- C1: MPN (none) -> C2012C0G1H103K060AA; PartNum C2012C0G1H103K060AA -> (none)
- C2, C3: MPN (none) -> GRM32ER71J106KA12L; PartNum GRM32ER71J106KA12L -> (none)
- C4: MPN (none) -> C0805C104M5RACTU; PartNum C0805C104M5RACTU -> (none)
- C5: MPN (none) -> GRM32ER61C476KE15L; PartNum GRM32ER61C476KE15L -> (none)
- D1, D2: MPN (none) -> PMEG6010CEH,115; PartNum PMEG6010CEH,115 -> (none)
- J1, J2: MPN (none) -> MJEA-660X1XXX; Manufacturer (none) -> Wayconn
- J3: MPN (none) -> PZ254V-11-04P; Manufacturer (none) -> XFCN
- J4: MPN (none) -> DILB24P-223TLF; Manufacturer (none) -> Amphenol ICC (FCI)
- L1: MPN (none) -> NPI105C121MTRF or SRR1050A-121Y; Manufacturer NIC Components -> NIC Components or Bournes Inc.; PartNum NPI105C121MTRF -> (none)
- Q1: MPN (none) -> MMBT3904; Manufacturer (none) -> Guangdong Hottech
- R1, R2: MPN (none) -> RC0603FR-07100KL; PartNum RC0603FR-07100KL -> (none)
- R3: MPN (none) -> RC0603FR-07470RL; PartNum RC0603FR-07470RL -> (none)
- R4, R5: MPN (none) -> RC0603FR-0710KL; PartNum RC0603FR-0710KL -> (none)
- U1: MPN (none) -> LM2678S-5.0/NOPB; PartNum LM2678S-5.0/NOPB -> (none)
Changed lines of the file:
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@@
 			)
 		)
-		(property "PartNum" "PMEG6010CEH,115"
+		(property "MPN" "PMEG6010CEH,115"
 			(at 132.08 57.15 0)
 			(effects
@@
 			)
 		)
-		(property "PartNum" "RC0603FR-07100KL"
+		(property "MPN" "RC0603FR-07100KL"
 			(at 93.98 123.19 0)
 			(effects
@@
 			)
 		)
-		(property "PartNum" "NPI105C121MTRF"
+		(property "MPN" "NPI105C121MTRF or SRR1050A-121Y"
 			(at 138.43 62.23 0)
 			(effects
@@
 			)
 		)
-		(property "Manufacturer" "NIC Components"
+		(property "Manufacturer" "NIC Components or Bournes Inc."
 			(at 138.43 62.23 0)
 			(effects
@@
 			)
 		)
-		(property "PartNum" "GRM32ER71J106KA12L"
+		(property "MPN" "GRM32ER71J106KA12L"
 			(at 87.63 64.77 90)
 			(effects
@@
 			)
 		)
+		(property "Manufacturer" "Guangdong Hottech"
+			(at 128.27 132.08 0)
+			(effects
+				(font
+					(size 1.27 1.27)
+				)
+				(hide yes)
+			)
+		)
+		(property "MPN" "MMBT3904"
+			(at 128.27 132.08 0)
+			(effects
+				(font
+					(size 1.27 1.27)
+				)
+				(hide yes)
+			)
+		)
 		(pin "2"
 		)
@@
 			)
 		)
-		(property "PartNum" "LM2678S-5.0/NOPB"
+		(property "MPN" "LM2678S-5.0/NOPB"
 			(at 85.09 36.83 0)
 			(effects
@@
 			)
 		)
-		(property "PartNum" "RC0603FR-07100KL"
+		(property "MPN" "RC0603FR-07100KL"
 			(at 93.98 101.6 0)
 			(effects
@@
 			)
 		)
-		(property "PartNum" "C2012C0G1H103K060AA"
+		(property "MPN" "C2012C0G1H103K060AA"
 			(at 64.77 39.37 0)
 			(effects
@@
 			)
 		)
+		(property "Manufacturer" "Amphenol ICC (FCI)"
+			(at 149.86 96.52 0)
+			(effects
+				(font
+					(size 1.27 1.27)
+				)
+				(hide yes)
+			)
+		)
+		(property "MPN" "DILB24P-223TLF"
+			(at 149.86 96.52 0)
+			(effects
+				(font
+					(size 1.27 1.27)
+				)
+				(hide yes)
+			)
+		)
 		(pin "19"
 		)
@@
 			)
 		)
+		(property "Manufacturer" "XFCN"
+			(at 119.38 109.22 0)
+			(effects
+				(font
+					(size 1.27 1.27)
+				)
+				(hide yes)
+			)
+		)
+		(property "MPN" "PZ254V-11-04P"
+			(at 119.38 109.22 0)
+			(effects
+				(font
+					(size 1.27 1.27)
+				)
+				(hide yes)
+			)
+		)
 		(pin "2"
 		)
@@
 			)
 		)
-		(property "PartNum" "RC0603FR-0710KL"
+		(property "MPN" "RC0603FR-0710KL"
 			(at 138.43 109.22 0)
 			(effects
@@
 			)
 		)
-		(property "Datasheet" "~"
+		(property "Datasheet" "https://www.wayconn.com/rj25-6p6c-pcb-mount-ra/"
 			(at 48.26 130.175 90)
 			(effects
@@
 			)
 		)
+		(property "Manufacturer" "Wayconn"
+			(at 48.26 130.81 0)
+			(effects
+				(font
+					(size 1.27 1.27)
+				)
+				(hide yes)
+			)
+		)
+		(property "MPN" "MJEA-660X1XXX"
+			(at 48.26 130.81 0)
+			(effects
+				(font
+					(size 1.27 1.27)
+				)
+				(hide yes)
+			)
+		)
 		(pin "5"
 		)
@@
 			)
 		)
-		(property "PartNum" "GRM32ER61C476KE15L"
+		(property "MPN" "GRM32ER61C476KE15L"
 			(at 132.08 73.66 90)
 			(effects
@@
 			)
 		)
-		(property "PartNum" "RC0603FR-0710KL"
+		(property "MPN" "RC0603FR-0710KL"
 			(at 138.43 138.43 0)
 			(effects
@@
 			)
 		)
-		(property "PartNum" "PMEG6010CEH,115"
+		(property "MPN" "PMEG6010CEH,115"
 			(at 77.47 82.55 0)
 			(effects
@@
 			)
 		)
-		(property "PartNum" "C0805C104M5RACTU"
+		(property "MPN" "C0805C104M5RACTU"
 			(at 87.63 57.15 90)
 			(effects
@@
 			)
 		)
-		(property "PartNum" "RC0603FR-07470RL"
+		(property "MPN" "RC0603FR-07470RL"
 			(at 105.41 123.19 0)
 			(effects
@@
 			)
 		)
-		(property "PartNum" "GRM32ER71J106KA12L"
+		(property "MPN" "GRM32ER71J106KA12L"
 			(at 87.63 72.39 90)
 			(effects
@@
 			)
 		)
-		(property "Datasheet" "~"
+		(property "Datasheet" "https://www.wayconn.com/rj25-6p6c-pcb-mount-ra/"
 			(at 48.26 98.425 90)
 			(effects
@@
 			(at 48.26 99.06 0)
 			(effects
+				(font
+					(size 1.27 1.27)
+				)
+				(hide yes)
+			)
+		)
+		(property "Manufacturer" "Wayconn"
+			(at 48.26 99.06 0)
+			(effects
+				(font
+					(size 1.27 1.27)
+				)
+				(hide yes)
+			)
+		)
+		(property "MPN" "MJEA-660X1XXX "
+			(at 48.26 99.06 0)
+			(effects
