File: PoolController.kicad_pcb (KiCad board)
At the start: 2 copper layers, 80 x 75 mm, 23 parts, among them J1 RJ12, J2 RJ12, J3 Header, J4 Conn_02x12_Counter_Clockwise, Q1 MMBT3904, U1 LM2678S-5.0/NOPB

Commit message: ### Fixed - Rev 14 - Fixed TX circuit to handle 12v as well as 7v
Parts:
- removed the R3 at (97.5, 97.5)
- R3: renamed from R4; value R10k -> R1k
- R4: renamed from R5; value R10k -> R100k
Connections:
- Q1 pad 3: Net-(Q1-C) -> Net-(J3-Pin_3)
Routing:
- net Net-(J3-Pin_3): track 66.7 -> 74.3 mm
- net Net-(Q1-C): track 5.94 -> 0.00 mm
Other:
- board text added: "J3 Header: * Power: ~24-40v * Data RX: 0 - 3.5v * Data TX: 0 - 12v * GND"
- board text removed: "J3 Header: * Power: ~24-40v * Data RX: 0 - 3.5v * Data TX: 0 - 7v * GND"
