File: PoolController.kicad_pcb (KiCad board)
At the start: 2 copper layers, 80 x 75 mm, 24 parts, among them J1 RJ12, J2 RJ12, J3 Header, J4 SSW-109-01-T-S, J5 SSW-109-01-T-S, Q1 MMBT3904, U1 LM2678S-5.0/NOPB

Commit message: Clean up track and update to rev16
Parts:
- moved D3 3.24 mm to (97.5, 70.9), turned to 90 degrees
Routing:
- net /+3V3_MODULE: track 32.0 -> 24.9 mm
- net /RX: track 57.7 -> 55.0 mm
