File: PoolController.kicad_sch (KiCad schematic)
At the start: 19 parts, among them J1 RJ12, J2 RJ12, J3 Header, J4 Conn_02x12_Counter_Clockwise, Q1 MMBT3904, U1 LM2678S-5.0/NOPB

Commit message: ### Fixed - Rev 14 - Fixed TX circuit to handle 12v as well as 7v
Parts:
- removed R3: R470, Resistor_SMD:R_0603_1608Metric, symbol Device:R
- R3: renamed from R4; value R10k -> R1k; MPN RC0603FR-0710KL -> RC0603FR-071KL
- R4: renamed from R5; value R10k -> R100k; MPN RC0603FR-0710KL -> RC0603FR-07100KL
Connections:
- net at Q1.3 (C): now also J1.4, J2.4, J3.3 (Pin_3), R1.1
Changed lines of the file:
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@@
 	(title_block
 		(title "Connect 10 Controller")
-		(date "2026-04-01")
-		(rev "13")
+		(date "2026-08-01")
+		(rev "14")
 	)
 	(text "+5v"
@@
 	(wire
 		(pts
-			(xy 105.41 119.38) (xy 105.41 111.76)
+			(xy 105.41 111.76) (xy 105.41 127)
 		)
 		(stroke
@@
 		(dnp no)
 		(fields_autoplaced yes)
-		(property "Reference" "R4"
+		(property "Reference" "R3"
 			(at 140.97 107.9499 0)
 			(effects
@@
 			)
 		)
-		(property "Value" "R10k"
+		(property "Value" "R1k"
 			(at 140.97 110.4899 0)
 			(effects
@@
 			)
 		)
-		(property "MPN" "RC0603FR-0710KL"
+		(property "MPN" "RC0603FR-071KL"
 			(at 138.43 109.22 0)
 			(effects
@@
 			(project "PoolController"
 				(path "/19c01251-b544-42b5-958c-1f3f3624b74e"
-					(reference "R4")
+					(reference "R3")
 					(unit 1)
 				)
@@
 		(dnp no)
 		(fields_autoplaced yes)
-		(property "Reference" "R5"
+		(property "Reference" "R4"
 			(at 140.97 137.1599 0)
 			(effects
@@
 			)
 		)
-		(property "Value" "R10k"
+		(property "Value" "R100k"
 			(at 140.97 139.6999 0)
 			(effects
@@
 			)
 		)
-		(property "MPN" "RC0603FR-0710KL"
+		(property "MPN" "RC0603FR-07100KL"
 			(at 138.43 138.43 0)
 			(effects
@@
 			(project "PoolController"
 				(path "/19c01251-b544-42b5-958c-1f3f3624b74e"
-					(reference "R5")
+					(reference "R4")
 					(unit 1)
 				)
@@
 					(unit 1)
 				)
-			)
-		)
-	)
-	(symbol
-		(lib_id "Device:R")
-		(at 105.41 123.19 0)
-		(unit 1)
-		(exclude_from_sim no)
-		(in_bom yes)
-		(on_board yes)
-		(dnp no)
-		(fields_autoplaced yes)
-		(property "Reference" "R3"
-			(at 107.95 121.9199 0)
-			(effects
-				(font
-					(size 1.27 1.27)
-				)
-				(justify left)
-			)
-		)
-		(property "Value" "R470"
-			(at 107.95 124.4599 0)
-			(effects
-				(font
-					(size 1.27 1.27)
-				)
-				(justify left)
-			)
-		)
-		(property "Footprint" "Resistor_SMD:R_0603_1608Metric"
-			(at 103.632 123.19 90)
-			(effects
-				(font
-					(size 1.27 1.27)
-				)
-				(hide yes)
-			)
-		)
-		(property "Datasheet" "~"
-			(at 105.41 123.19 0)
-			(effects
-				(font
-					(size 1.27 1.27)
-				)
-				(hide yes)
-			)
-		)
-		(property "Description" "Resistor"
-			(at 105.41 123.19 0)
-			(effects
-				(font
-					(size 1.27 1.27)
-				)
-				(hide yes)
-			)
-		)
-		(property "MPN" "RC0603FR-07470RL"
-			(at 105.41 123.19 0)
-			(effects
-				(font
-					(size 1.27 1.27)
-				)
-				(hide yes)
-			)
-		)
-		(property "Manufacturer" "YAGEO"
-			(at 105.41 123.19 0)
-			(effects
-				(font
-					(size 1.27 1.27)
-				)
-				(hide yes)
-			)
-		)
-		(pin "1"
-		)
-		(pin "2"
-		)
-		(instances
-			(project ""
-				(path "/19c01251-b544-42b5-958c-1f3f3624b74e"
-					(reference "R3")
-					(unit 1)
-				)
